File: ASD2101.sch (EAGLE design)
At the start: 15 parts, among them J1 20021111, J2 DF12-32-DS, J3 47346-0001, J4 DF12-32-DP, Q1 DMP2035U, U1 FT232RQ

Commit message: Updated to Rev4
Parts:
- added R4, R6: 0.0, tinycircuits:AS-ITM-000760402_SHORT
- added R5: 0.0, tinycircuits:AS-ITM-00076
Connections:
- removed net N$1: C4.1, U1.3V3OUT
- new net 3V3OUT: C4.1, R5.1, U1.3V3OUT
- new net N$4: Q1.D, R4.2, R5.2
- new net RTS: R6.1, U1.RTS
- net RSV2: now also R6.2
- net USBVCC: now also R4.1; no longer Q1.D
Other:
- note added: "3.3V Out: Pop R5 (50mA Max)"
- note added: "4"
- note added: "5V Out: Pop R4 (Default)"
- note added: "USB Power Option:"
- note removed: "3"
- moved on the sheet: Q1, R3

Commit message: Updated to Rev 6
Parts:
- removed U1: FT232RQ, tinycircuits:AS-ITM-00029
- added C5, C6: 47pF, tinycircuits:AS-ITM-00241
- added R10, R7, R8, R9: 27.0, tinycircuits:AS-ITM-00240
- added R11, R12: 1.00K, tinycircuits:AS-ITM-00003
- added U2: FT231XQ-R, tinycircuits:AS-ITM-00223
- J1: value 20021111 -> 47346-0001; device tinycircuits:AS-ITM-00022 -> tinycircuits:AS-ITM-00021; DNP T -> (none); PARTNO (none) -> AS-ITM-00021
- R4: device tinycircuits:AS-ITM-000760402_SHORT -> tinycircuits:AS-ITM-00076; VALUE (none) -> 0.0
Connections:
- removed net N$13: J3.3, U1.USBDP
- new net N$1: J3.2, R7.1
- new net N$10: R12.2, U2.TXD
- new net N$3: J1.3, R10.1
- new net N$8: J3.3, R8.1
- new net N$9: R11.2, U2.RXD
- new net USBDM: C5.1, R7.2, R9.2, U2.USBDM
- new net USBDP: C6.1, R10.2, R8.2, U2.USBDP
- net 3V3OUT: now also R1.2, R2.2, U2.3V3OUT, U2.RESET, U2.VCCIO; no longer U1.3V3OUT
- net DTR: now also U2.DTR; no longer U1.DTR
- net GND: now also C5.2, C6.2, J1.5, J1.P1, J1.P2, J1.P3, J1.P4, J1.P5, J1.P6, U2.GND0, U2.GND1, U2.GND2; no longer J1.6, U1.AGND, U1.GND1, U1.GND2, U1.GND3, U1.PAD, U1.TEST
- net IO0: now also R12.1; no longer U1.TXD
- net IO1: now also R11.1; no longer U1.RXD
- net MISO: no longer J1.1
- net MOSI: no longer J1.4
- net N$16: now also U2.CBUS1; no longer U1.TXLED
- net N$2: now also J1.2, R9.1; no longer J3.2, U1.USBDM
- net N$5: now also U2.CBUS2; no longer U1.RXLED
- net RESET: no longer J1.5
- net RTS: now also U2.RTS; no longer U1.RTS
- net SCK: no longer J1.3
- net USBVCC: now also J1.1, U2.VCC; no longer U1.VCC
- net VCC: no longer J1.2, R1.2, R2.2, U1.VCCIO
Other:
- note added: "6"
- note removed: "4"
- note removed: "ICSP Connector"
- moved on the sheet: C1, C2, C3, C4, D1, D2, J3, R1, R2, R6
