File: design_files/ASD2101.brd (EAGLE design)
At the start: 22.5 x 21.3 mm, 27 parts, among them J1 47346-0001, J2 DF12-32-DS, J3 47346-0001, J4 DF12-32-DP, Q1 DMP2035U, U2 FT231XQ-R

Commit message: update format
Other:
- board text added: "TinyCircuits.com"
- board text removed: "Tiny-Circuits.com"
- board text removed: "TinyShield - USB & ICP"
Changed lines of the file:
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@@
 <setting verticaltext="up"/>
 </settings>
-<grid distance="7" unitdist="mil" unit="mm" style="lines" multiple="1" display="yes" altdistance="0.025" altunitdist="inch" altunit="inch"/>
+<grid distance="0.1" unitdist="mm" unit="mm" style="lines" multiple="1" display="yes" altdistance="0.025" altunitdist="inch" altunit="inch"/>
 <layers>
 <layer number="1" name="Top" color="4" fill="1" visible="yes" active="yes"/>
@@
 <wire x1="0" y1="50.8" x2="0" y2="0" width="0.127" layer="48"/>
 <dimension x1="10" y1="30" x2="30" y2="30" x3="20" y3="33.454653125" layer="48"/>
-<text x="48.111025" y="4.365003125" size="0.889" layer="48">TinyShield - USB &amp; ICP</text>
+<text x="48.111025" y="4.365003125" size="0.889" layer="48">USB TinyShield</text>
 <text x="44.986825" y="1.7714" size="0.889" layer="48">AS-PCB-ASD2101</text>
 <text x="67.3810375" y="1.6952" size="0.889" layer="48">6</text>
@@
 <rectangle x1="17.87298125" y1="25.08461875" x2="18.09141875" y2="25.08969375" layer="22"/>
 <rectangle x1="17.89838125" y1="25.089696875" x2="18.0609375" y2="25.094778125" layer="22"/>
-<text x="14.573203125" y="21.747828125" size="0.762" layer="22" rot="MR180">Tiny-Circuits.com</text>
+<text x="15.106603125" y="21.747828125" size="0.762" layer="22" rot="MR180">TinyCircuits.com</text>
 <text x="15.04564375" y="19.51770625" size="0.762" layer="22" rot="MR180">ASD2101 - Rev6</text>
 <text x="15.37838125" y="20.604828125" size="0.762" layer="22" rot="MR180">USB TinyShield</text>
@@
 <element name="J3" library="tinycircuits" package="MICRO_USB" value="47346-0001" x="13" y="20.5">
 <attribute name="PARTNO" value="AS-ITM-00021" x="13" y="30.5" size="1.778" layer="27" display="off"/>
+<attribute name="PNPROTATION" value="90" x="13" y="20.5" size="1.778" layer="27" display="off"/>
 </element>
 <element name="C3" library="tinycircuits" package="C0603" value="10uF" x="25.0518" y="26.258" rot="R90">
@@
 <attribute name="PARTNO" value="AS-ITM-00026" x="29" y="21.95" size="1.778" layer="27" rot="R180" display="off"/>
 <attribute name="VALUE" value="AMBER" x="29" y="21.95" size="1.778" layer="27" rot="R180" display="off"/>
+<attribute name="PNPROTATION" value="90" x="29" y="21.95" size="1.778" layer="27" rot="R180" display="off"/>
 </element>
 <element name="D2" library="tinycircuits" package="LNJ_LED" value="AMBER" x="29" y="24.6" rot="R180">
 <attribute name="PARTNO" value="AS-ITM-00026" x="29" y="24.6" size="1.778" layer="27" rot="R180" display="off"/>
 <attribute name="VALUE" value="AMBER" x="29" y="24.6" size="1.778" layer="27" rot="R180" display="off"/>
+<attribute name="PNPROTATION" value="90" x="29" y="24.6" size="1.778" layer="27" rot="R180" display="off"/>
 </element>
 <element name="Q1" library="tinycircuits" package="SOT23" value="DMP2035U" x="27.9894" y="14.6524" rot="R270">
 <attribute name="PARTNO" value="AS-ITM-00024" x="27.9894" y="14.6524" size="1.778" layer="27" rot="R270" display="off"/>
 <attribute name="VALUE" value="DMP2035U" x="27.9894" y="14.6524" size="1.778" layer="27" rot="R270" display="off"/>
+<attribute name="PNPROTATION" value="0" x="27.9894" y="14.6524" size="1.778" layer="27" rot="R270" display="off"/>
 </element>
 <element name="U$1" library="tinycircuits" package="DOCFIELD-TINYCIRCUITS-PCB" value="" x="43.9674" y="-0.0254">
@@
 <attribute name="PARTNO" value="AS-ITM-00223" x="23.8" y="21" size="1.778" layer="27" rot="R270" display="off"/>
 <attribute name="VALUE" value="FT231XQ-R " x="23.8" y="21" size="1.778" layer="27" rot="R270" display="off"/>
+<attribute name="PNPROTATION" value="270" x="23.8" y="21" size="1.778" layer="27" rot="R270" display="off"/>
 </element>
 <element name="R7" library="tinycircuits" package="0402" value="27.0" x="18.55" y="19.8">
 <attribute name="VALUE" value="27.0" x="18.55" y="19.8" size="1.778" layer="27" display="off"/>
-<attribute name="PARNTO" value="AS-ITM-00240" x="18.55" y="19.8" size="1.778" layer="27" display="off"/>
+<attribute name="PARTNO" value="AS-ITM-00240" x="18.55" y="19.8" size="1.778" layer="27" display="off"/>
 </element>
 <element name="R8" library="tinycircuits" package="0402" value="27.0" x="17.5" y="21.35" rot="R90">
 <attribute name="VALUE" value="27.0" x="17.5" y="21.35" size="1.778" layer="27" rot="R90" display="off"/>
-<attribute name="PARNTO" value="AS-ITM-00240" x="17.5" y="21.35" size="1.778" layer="27" rot="R90" display="off"/>
+<attribute name="PARTNO" value="AS-ITM-00240" x="17.5" y="21.35" size="1.778" layer="27" rot="R90" display="off"/>
 </element>
 <element name="C5" library="tinycircuits" package="0402" value="47pF" x="19.95" y="19.1" rot="R270">
@@
 <attribute name="PARTNO" value="AS-ITM-00021" x="28.5" y="32.8" size="1.778" layer="27" rot="R270" display="off"/>
 <attribute name="VALUE" value="47346-0001" x="28.5" y="32.8" size="1.778" layer="27" rot="R270" display="off"/>
+<attribute name="PNPROTATION" value="90" x="20" y="27" size="1.778" layer="27" rot="R270" display="off"/>
 </element>
 <element name="R9" library="tinycircuits" package="0402" value="27.0" x="20.35" y="21.15" rot="R270">
 <attribute name="VALUE" value="27.0" x="29.35" y="29.05" size="1.778" layer="27" rot="R270" display="off"/>
-<attribute name="PARNTO" value="AS-ITM-00240" x="20.35" y="21.15" size="1.778" layer="27" rot="R270" display="off"/>
+<attribute name="PARTNO" value="AS-ITM-00240" x="20.35" y="21.15" size="1.778" layer="27" rot="R270" display="off"/>
 </element>
 <element name="R10" library="tinycircuits" package="0402" value="27.0" x="18.95" y="22.85" rot="R180">
 <attribute name="VALUE" value="27.0" x="29.05" y="15.45" size="1.778" layer="27" rot="R180" display="off"/>
-<attribute name="PARNTO" value="AS-ITM-00240" x="18.95" y="22.85" size="1.778" layer="27" rot="R180" display="off"/>
+<attribute name="PARTNO" value="AS-ITM-00240" x="18.95" y="22.85" size="1.778" layer="27" rot="R180" display="off"/>
 </element>
 <element name="R11" library="tinycircuits" package="0402" value="1.00K" x="11.85" y="14.4" rot="R90">
