File: design_files/ASD2101.sch (EAGLE design)
At the start: 26 parts, among them J1 47346-0001, J2 DF12-32-DS, J3 47346-0001, J4 DF12-32-DP, Q1 DMP2035U, U2 FT231XQ-R

Commit message: update format
Other:
- note added: "FTDI FT231 USB to Serial Converter"
- note added: "Hand Populated: -"
- note added: "Hand Soldered: -"
- note added: "Micro USB - Side"
- note added: "Micro USB - Top"
- note added: "Non Populated: J1, R5, R6, R9, R10"
- note added: "Non Populated: J3, R5, R6, R7, R8"
- note added: "Power Jumpers and 5V Switch"
- note added: "USB TinyShield"
- note added: "Variant: Side - R"
- note added: "Variant: Top - R-T"
- note removed: "Micro USB"
- note removed: "TinyShield - USB & ICP"
- moved on the sheet: C1, C2, C3, C4, C5, C6, D1, D2, J1, J3, Q1, R1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
